File: pcb_files/ModuloSlave.sch (EAGLE design)
At the start: 77 parts, among them IC1 MEGA8-P, IC2 7805T, J1 JumpersSerie

Commit message: Modulo expansão
*faltam ligações
Parts:
- removed ALIMENTACAOOUT, OUT7, OUT8: (no value), con-ptr500:AK300/2
- removed BNTRESET: DTE6K, switch-misc:DTE6K
- removed COSC_MC_1, COSC_MC_2, CRESET, CVCC_MC, CVDD_MCP: (no value), SparkFun-Passives:CAP_
- removed DOUT1, DOUT2, DOUT3, DOUT4, DOUT5, DOUT6, DOUT7, DOUT8, DOUT9, DRX, DRX_MCP, DTX, DTX_MCP: HLMP6, display-hp:HLMP6
- removed IC1: MEGA8-P, atmel:MEGA8-P
- removed IC2: 7805T, linear:7805T
- removed IN1, IN2, IN3, IN4, IN5, IN6, IN7, OPTOUT1, OPTOUT2: LTV816, optocoupler:LTV816
- removed J1: JumpersSerie, SAMTEC-BBx-ERx-SLx-SDL_By_element14_Batch_1:BBS-105-G-A
- removed JP1, JP2: (no value), pinhead:PINHD-1X6
- removed MCP_RX, MCP_TX, R13, R14, R15, R16, R17, R18, R19: (no value), resistor:R-EU_0204/7
- removed OSC_MC: (no value), crystal:CRYSTALHC49S
- removed RCAN, RRESET, RRESET_MCP, RRX, RTX, RVCC_MC: (no value), rcl:L-EU0204V
- added ALIMENTACAO, LINHASCANOUT, X1, X2: (no value), con-ptr500:AK300/2
- added CVDD_25015, CVDD_2551: (no value), SparkFun-Passives:CAP_
- added D1, D2, D3, D7: HLMP6, display-hp:HLMP6
- added LED1, LED2, LED3, LED4: (no value), eagle-ltspice:LED_E
- added OK1, OK2, OKOUT1, OKOUT2, OKOUT3, OKOUT4, OKOUT5, OKOUT6: LTV816, optocoupler:LTV816
- added RVSS_2551: (no value), rcl:L-EU0204V
- R1, R10, R11, R12, R2, R3, R4, R5, R6, R7, R8, R9: device resistor:R-EU_0204/7 -> resistor:R-EU_0204/5
- U$3: value MCP2515-I/P -> MCP25050-E/P; device Microchip_By_element14_Batch_1:MCP2515-I/P -> Microchip_By_element14_Batch_1:MCP25050-E/P
- U$4: value MCP2551-I/P -> MCP2551-E/P; device Microchip_By_element14_Batch_1:MCP2551-I/P -> Microchip_By_element14_Batch_1:MCP2551-E/P
Connections:
- removed net MISO: IC1.PB4(MISO), JP2.5, U$3.SO
- removed net MOSI: IC1.PB3(MOSI/OC2), JP2.4, U$3.SI
- removed net N$20: IN1.C, OUT5-2.KL
- removed net N$27: IC1.PC3(ADC3), JP1.4
- removed net N$31: IN2.EMIT, IN3.EMIT, R5.1, R7.2
- removed net N$35: DOUT6.A, R6.1
- removed net N$36: DOUT7.A, R7.1
- removed net N$37: IN5.COL
- removed net N$38: IN5.EMIT, R12.2, R13.2
- removed net N$39: DOUT3.A, R13.1
- removed net N$40: OUT8-1.KL, R8.2
- removed net N$41: IN4.A, R8.1
- removed net N$42: IN4.C, OUT8-2.KL
- removed net N$43: IN4.COL
- removed net N$44: IN4.EMIT, R10.1, R9.1
- removed net N$45: DOUT9.A, R10.2
- removed net N$46: IN6.COL
- removed net N$47: IN6.EMIT, R15.2, R16.2
- removed net N$48: DOUT4.A, R16.1
- removed net N$49: OUT7-1.KL, R17.2
- removed net N$50: IN7.A, R17.1
- removed net N$51: IN7.C, OUT7-2.KL
- removed net N$52: IN7.COL
- removed net N$53: IN7.EMIT, R18.1, R19.1
- removed net N$54: DOUT8.A, R19.2
- removed net PB0: IC1.PB0(ICP), JP2.1
- removed net PB1: IC1.PB1(OC1A), JP2.2
- removed net PD2: IC1.PD2(INT0), JP3.3
- removed net PD3: IC1.PD3(INT1), JP3.4, OPTOUT2.A
- removed net PD4: IC1.PD4(XCK/T0), JP3.5, OPTOUT1.A
- removed net PD5: IC1.PD5(T1), JP3.6
- removed net PD6: IC1.PD6(AIN0), JP3.7
- removed net PD7: IC1.PD7(AIN1), JP3.8
- removed net RST: CRESET.2, J1.5
- removed net RXCAN: DTX_MCP.K, U$3.RXCAN, U$4.RXD
- removed net RXD: DRX.A, IC1.PD0(RXD), J1.4, JP3.1
- removed net SCK: IC1.PB5(SCK), JP2.6, U$3.SCK
- removed net SS: IC1.PB2(SS/OC1B), JP2.3, U$3.~CS
- removed net TXCAN: DRX_MCP.K, U$3.TXCAN, U$4.TXD
- removed net TXD: DTX.A, IC1.PD1(TXD), J1.3, JP3.2
- new net GP0: JP3.1, OKOUT1.A, U$3.GP0/AN0
- new net GP1: JP3.2, OKOUT2.A, U$3.GP1/AN1
- new net GP2: JP3.3, OKOUT3.A, U$3.GP2/AN2/PWM1
- new net GP4: JP3.5, OKOUT4.A, U$3.GP4/VREF-
- new net GP5: JP3.6
- new net GP6: JP3.7
- new net IA: JP3.8, U$3.GP7/~RST/VPP
- new net IB: JP3.4, U$3.GP3/AN3/PWM2
- new net N3: OUT5-2.KL
- new net OUT3+: OKOUT3.COL, OUT3-1.KL
- new net OUT3-: OKOUT3.EMIT, OUT3-2.KL
- new net OUT4+: OKOUT4.COL, OUT4-1.KL
- new net OUT4-: OKOUT4.EMIT, OUT4-2.KL
- new net OUT5+: OUT6-2.KL
- new net OUT5-: OUT5-1.KL
- new net OUT6-: OUT6-1.KL
- new net RX: U$3.RXCAN, U$4.RXD
- new net TX: U$3.TXCAN, U$4.TXD
- net 5V: now also OK1.COL, OK2.COL; no longer IC2.VO, IN1.COL, IN2.COL, IN3.COL, MCP_RX.2, MCP_TX.2, R1.2
- net CANH: now also LINHASCANOUT-1.KL; no longer RCAN.2
- net CANL: now also LINHASCANOUT-2.KL; no longer RCAN.1
- net GND: now also ALIMENTACAO-1.KL, CVDD_25015.1, CVDD_2551.1, LED1.C, LED2.C, R10.2, R11.2, R12.2, R3.1, R5.1, R7.2, R8.2, RVSS_2551.1; no longer ALIMENTACAOOUT-1.KL, BNTRESET.S, COSC_MC_1.1, COSC_MC_2.1, CVCC_MC.2, CVDD_MCP.2, DOUT1.K, DOUT2.K, DOUT3.K, DOUT4.K, DOUT5.K, DOUT6.K, DOUT7.K, DOUT8.K, DOUT9.K, IC1.GND, IC1.GND@1, IC2.GND, J1.2, R12.1, R15.1, R18.2, R4.2, R5.2, RRX.1, RTX.1, U$4.VSS
- net N$1: now also D7.A, OKOUT1.C; no longer DOUT2.A, OPTOUT2.C
- net N$10: now also RVSS_2551.2, U$4.VSS; no longer OUT5-1.KL, R2.2
- net N$11: now also OK2.EMIT, R5.2, R6.2; no longer IN1.A, R2.1
- net N$12: now also OK1.EMIT, R3.2, R4.2; no longer IN5.C, OUT3-2.KL
- net N$13: now also U$3.OSC1/CLKIN; no longer U$3.OSC1
- net N$15: now also LED1.A, R4.1; no longer OUT4-1.KL, R14.2
- net N$16: now also LED2.A, R6.1; no longer IN6.A, R14.1
- net N$17: now also OK2.A, R2.2; no longer IN6.C, OUT4-2.KL
- net N$18: now also R2.1, X2-1.KL; no longer DTX.K, RTX.2
- net N$19: now also OK2.C, X2-2.KL; no longer DRX.K, RRX.2
- net N$2: now also D1.A, OKOUT3.C; no longer DOUT1.A, OPTOUT1.C
- net N$21: now also OKOUT5.A; no longer OUT6-1.KL, R3.2
- net N$22: now also OKOUT6.A; no longer RRESET_MCP.2, U$3.~RESET
- net N$23: now also LED3.C, R11.1; no longer IC1.AVCC, RVCC_MC.2
- net N$24: now also D2.A, OKOUT2.C; no longer IC1.PC0(ADC0), JP1.1
- net N$25: now also OKOUT5.COL; no longer IC1.PC1(ADC1), JP1.2
- net N$26: now also LED4.C, R12.1; no longer IC1.PC2(ADC2), JP1.3
- net N$28: now also LED4.A, OKOUT6.C; no longer IC1.PC4(ADC4/SDA), JP1.5
- net N$29: now also OKOUT5.EMIT; no longer IC1.PC5(ADC5/SCL), JP1.6
- net N$3: now also D7.K, R9.1; no longer COSC_MC_2.2, IC1.PB7(XTAL2/TOSC2), OSC_MC.1
- net N$30: now also LED3.A, OKOUT5.C; no longer IN1.EMIT, R4.1, R6.2
- net N$32: now also OKOUT6.COL; no longer IN2.A, IN3.A, R3.1
- net N$33: now also D3.A, OKOUT4.C; no longer IN2.C, IN3.C, OUT6-2.KL
- net N$34: now also OKOUT6.EMIT; no longer DOUT5.A, R1.1
- net N$4: now also D1.K, R7.1; no longer COSC_MC_1.2, IC1.PB6(XTAL1/TOSC1), OSC_MC.2
- net N$5: now also D2.K, R8.1; no longer OUT3-1.KL, R11.1
- net N$6: now also D3.K, R10.1; no longer DRX_MCP.A, MCP_RX.1
- net N$7: now also OK1.A, R1.2; no longer DTX_MCP.A, MCP_TX.1
- net N$8: now also R1.1, X1-1.KL; no longer IN5.A, R11.2
- net N$9: now also OK1.C, X1-2.KL; no longer BNTRESET.P@1, CRESET.1, IC1.PC6(/RESET), RRESET.2
- net OUT1+: now also OKOUT1.COL; no longer OPTOUT1.COL
- net OUT1-: now also OKOUT1.EMIT; no longer OPTOUT1.EMIT
- net OUT2+: now also OKOUT2.COL; no longer OPTOUT2.COL
- net OUT2-: now also OKOUT2.EMIT; no longer OPTOUT2.EMIT
- net VCC: now also ALIMENTACAO-2.KL, CVDD_25015.2, CVDD_2551.2; no longer ALIMENTACAOOUT-2.KL, CVCC_MC.1, CVDD_MCP.1, IC1.VCC@1, IC2.VI, J1.1, RRESET.1, RRESET_MCP.1, RVCC_MC.1, U$3.~INT
Other:
- note added: "Linhas CAN saida"
- note removed: "Linhas Serie"
- note removed: "Regulador de tensão"
- moved on the sheet: COSC_MCP_1, COSC_MCP_2, JP3, LINHASCAN-1, LINHASCAN-2, OSC_MCP, OUT1-1, OUT1-2, OUT2-1, OUT2-2, OUT3-1, OUT3-2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
