File: pcb_files/ModuloMaster.sch (EAGLE design)
At the start: 77 parts, among them IC1 MEGA8-P, IC2 7805T, J1 JumpersSerie

Commit message: Fix some issues in Master and Slave module
Fix some issues.
Frist broad for Master module.
Parts:
- removed ALIMENTACAOOUT, LINHASCAN, OUT4, OUT5, OUT6, OUT7, OUT8: (no value), con-ptr500:AK300/2
- removed BNTRESET: DTE6K, switch-misc:DTE6K
- removed COSC_MC_1, COSC_MC_2, CRESET, CVCC_MC, CVDD_MCP: (no value), SparkFun-Passives:CAP_
- removed DOUT8, DRX, DTX: HLMP6, display-hp:HLMP6
- removed IN1, IN2, IN3, IN4, IN5, IN6, IN7, OPTOUT1, OPTOUT2: LTV816, optocoupler:LTV816
- removed J1: JumpersSerie, SAMTEC-BBx-ERx-SLx-SDL_By_element14_Batch_1:BBS-105-G-A
- removed R19: (no value), resistor:R-EU_0204/7
- removed RCAN, RRESET, RRESET_MCP, RRX, RTX, RVCC_MC: (no value), rcl:L-EU0204V
- added ALIMENTACAO12V, ENT1, ENT2, ENT3, ENT4, ENT5: (no value), con-ptr500:AK300/2
- added C1, C3: (no value), rcl:C-EU025-025X050
- added C10, C6: (no value), SparkFun-Passives:CAP_
- added C2: (no value), rcl:CPOL-EUSANYO_C6
- added C4, C5: 22pF, SparkFun-Passives:CAP_
- added C7: 10u 35V, rcl:CPOL-EUSANYO_C6
- added D1: 1N4004, diode:1N4004
- added R20, R21: (no value), resistor:R-EU_0204/7
- added R22, R27: 10k, resistor:R-EU_0204/7
- added R24, R25, R26: 100k, resistor:R-EU_0204/7
- added R30: 47k, resistor:R-EU_0204/7
- added S1, S2, S3: (no value), SparkFun-Retired:TAC_SWITCHPTH
- added U$1, U$2, U$5, U$6, U$7, U$8, U$9: OPTO-RELAY-CPC1017N, Feesta-parts:OPTO-RELAY-CPC1017N
- MCP_RX, MCP_TX: value (none) -> 330
- R17: value (none) -> 10k
- R18: value (none) -> 120
Connections:
- net PB0 renamed N$56
- net PB1 renamed N$57
- net PD5 renamed N$66
- net PD6 renamed N$65
- net PD7 renamed N$64
- removed net N$18: DTX.K, RTX.2
- removed net N$19: DRX.K, RRX.2
- removed net N$24: IC1.PC0(ADC0), JP1.1
- removed net N$38: IN5.EMIT, R12.2, R13.2
- removed net N$43: IN4.COL
- removed net N$44: IN4.EMIT, R10.1, R9.1
- removed net N$46: IN6.COL
- removed net N$47: IN6.EMIT, R15.2, R16.2
- removed net N$49: OUT7-1.KL, R17.2
- removed net N$50: IN7.A, R17.1
- removed net N$51: IN7.C, OUT7-2.KL
- removed net N$52: IN7.COL
- removed net N$53: IN7.EMIT, R18.1, R19.1
- removed net N$54: DOUT8.A, R19.2
- removed net OUT1+: OPTOUT1.COL, OUT1-1.KL
- removed net OUT1-: OPTOUT1.EMIT, OUT1-2.KL
- removed net OUT2+: OPTOUT2.COL, OUT2-1.KL
- removed net OUT2-: OPTOUT2.EMIT, OUT2-2.KL
- removed net RST: CRESET.2, J1.5
- removed net RXD: DRX.A, IC1.PD0(RXD), J1.4, JP3.1
- removed net TXD: DTX.A, IC1.PD1(TXD), J1.3, JP3.2
- new net ADC0: IC1.PC0(ADC0), JP1.1, R4.1, R6.2, U$5.LOAD_2
- new net ADC1: IC1.PC1(ADC1), JP1.2, R5.1, R7.2, U$6.LOAD_2
- new net ADC2: IC1.PC2(ADC2), JP1.3, R10.1, R9.1, U$7.LOAD_2
- new net ADC3: IC1.PC3(ADC3), JP1.4, R12.2, R13.2, U$8.LOAD_2
- new net ADC4: IC1.PC4(ADC4/SDA), JP1.5, R15.2, R16.2, U$9.LOAD_2
- new net ADC5: IC1.PC5(ADC5/SCL), JP1.6, R17.2, S3.3, S3.4
- new net N$62: IC1.PD0(RXD), JP3.1
- new net N$63: IC1.PD1(TXD), JP3.2
- new net VDD: ALIMENTACAO12V-1.KL, C1.1, C7.+, D1.A, IC2.VI, U$1.LOAD_1, U$2.LOAD_1
- net 5V: now also C2.+, C3.1; no longer IN1.COL, IN2.COL, IN3.COL, MCP_RX.2, MCP_TX.2
- net CANH: now also OUT3-2.KL, R18.1; no longer LINHASCAN-1.KL, RCAN.2
- net CANL: now also OUT3-1.KL, R18.2; no longer LINHASCAN-2.KL, RCAN.1
- net GND: now also ALIMENTACAO12V-2.KL, C1.2, C10.1, C2.-, C3.2, C4.1, C5.1, C6.1, C7.-, D1.C, OUT1-2.KL, OUT2-2.KL, R20.2, R21.2, R30.2, S1.1, S1.2, S2.1, S2.2, S3.1, S3.2; no longer ALIMENTACAOOUT-1.KL, BNTRESET.S, COSC_MC_1.1, COSC_MC_2.1, CVCC_MC.2, CVDD_MCP.2, DOUT1.K, DOUT2.K, DOUT8.K, J1.2, R18.2, RRX.1, RTX.1, U$4.RS
- net N$1: now also U$2.CONTROL_-; no longer OPTOUT2.C
- net N$10: now also ENT1-1.KL; no longer OUT5-1.KL
- net N$11: now also U$5.CONTROL_+; no longer IN1.A
- net N$12: now also ENT4-2.KL, U$8.CONTROL_-; no longer IN5.C, OUT3-2.KL
- net N$15: now also ENT5-1.KL; no longer OUT4-1.KL
- net N$16: now also U$9.CONTROL_+; no longer IN6.A
- net N$17: now also ENT5-2.KL, U$9.CONTROL_-; no longer IN6.C, OUT4-2.KL
- net N$2: now also U$1.CONTROL_-; no longer OPTOUT1.C
- net N$20: now also ENT1-2.KL, U$5.CONTROL_-; no longer IN1.C, OUT5-2.KL
- net N$21: now also ENT2-1.KL; no longer OUT6-1.KL
- net N$22: now also OUT1-1.KL, U$1.LOAD_2; no longer RRESET_MCP.2, U$3.~RESET
- net N$23: now also IC1.PC6(/RESET), R22.2, S1.3, S1.4; no longer IC1.AVCC, RVCC_MC.2
- net N$25: now also DOUT1.K, R20.1; no longer IC1.PC1(ADC1), JP1.2
- net N$26: now also OUT2-1.KL, U$2.LOAD_2; no longer IC1.PC2(ADC2), JP1.3
- net N$27: now also DOUT2.K, R21.1; no longer IC1.PC3(ADC3), JP1.4
- net N$28: now also R30.1, U$4.RS; no longer IC1.PC4(ADC4/SDA), JP1.5
- net N$29: now also R25.1, U$3.~TX1RTS; no longer IC1.PC5(ADC5/SCL), JP1.6
- net N$3: now also C4.2; no longer COSC_MC_2.2
- net N$30: now also R24.1, U$3.~TX0RTS; no longer IN1.EMIT, R4.1, R6.2
- net N$31: now also R26.1, U$3.~TX2RTS; no longer IN2.EMIT, IN3.EMIT, R5.1, R7.2
- net N$32: now also ENT2-2.KL, U$6.CONTROL_-; no longer IN2.A, IN3.A, R3.1
- net N$33: now also R3.1, U$6.CONTROL_+; no longer IN2.C, IN3.C, OUT6-2.KL
- net N$37: now also R27.2, S2.3, S2.4, U$3.~RESET; no longer IN5.COL
- net N$4: now also C5.2; no longer COSC_MC_1.2
- net N$40: now also ENT3-1.KL; no longer OUT8-1.KL
- net N$41: now also U$7.CONTROL_+; no longer IN4.A
- net N$42: now also ENT3-2.KL, U$7.CONTROL_-; no longer IN4.C, OUT8-2.KL
- net N$5: now also ENT4-1.KL; no longer OUT3-1.KL
- net N$8: now also U$8.CONTROL_+; no longer IN5.A
- net N$9: now also C10.2, IC1.AREF; no longer BNTRESET.P@1, CRESET.1, IC1.PC6(/RESET), RRESET.2
- net PD2: now also U$3.~INT
- net PD3: now also U$1.CONTROL_+; no longer OPTOUT2.A
- net PD4: now also U$2.CONTROL_+; no longer OPTOUT1.A
- net VCC: now also C6.2, IC1.AVCC, MCP_RX.2, MCP_TX.2, R17.1, R22.1, R24.2, R25.2, R26.2, R27.1, U$5.LOAD_1, U$6.LOAD_1, U$7.LOAD_1, U$8.LOAD_1, U$9.LOAD_1; no longer ALIMENTACAOOUT-2.KL, CVCC_MC.1, CVDD_MCP.1, IC2.VI, J1.1, RRESET.1, RRESET_MCP.1, RVCC_MC.1, U$3.~INT
Other:
- note added: "ATMEGA328P"
- note added: "Linhas saída CAN"
- note added: "MCP2515 + MCP2551"
- note added: "Saídas"
- note removed: "Linhas CAN"
- note removed: "Linhas Serie"
- note removed: "Saidas"
- moved on the sheet: COSC_MCP_1, COSC_MCP_2, DOUT1, DOUT2, DOUT3, DOUT4, DOUT5, DOUT6, DOUT7, DOUT9, DRX_MCP, DTX_MCP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
